File: Donut of Doom/KiCad Files/Donut of Doom/Donut of Doom.kicad_pcb (KiCad board)
At the start: 2 copper layers, 25 x 53 mm, 43 parts, among them Q1 Q_NMOS_GSD, U3 H3LIS331DLTR

Commit message: Added 2nd accel, fixed mosfet, added more GND pads
Parts:
- removed the D5 at (153.9, 77.1)
- removed the EX1 at (141.8, 90.8)
- removed the EX2 at (141.8, 93.4)
- removed EX4: GP18, Battlebots:Pico_pth_pad
- removed the R4 at (149.6, 78.1)
- removed the R5 at (151.2, 78.0)
- removed the TP1 at (154.8, 86.2)
- removed the TP2 at (154.8, 81.9)
- added C3: 10uF, Capacitor_SMD:C_0805_2012Metric_Pad1.18x1.45mm_HandSolder, B.Cu at (146.5, 100.0)
- added C4: 0.1uF, Capacitor_SMD:C_0603_1608Metric_Pad1.08x0.95mm_HandSolder, B.Cu at (148.5, 99.2)
- added D6: GREEN ON LED, LED_SMD:LED_0603_1608Metric_Pad1.05x0.95mm_HandSolder, B.Cu at (154.3, 76.0)
- added D7: GREEN ON LED, LED_SMD:LED_0603_1608Metric_Pad1.05x0.95mm_HandSolder, B.Cu at (155.2, 100.5)
- added EX10: GND, Battlebots:Pico_pth_GND, F.Cu at (159.5, 101.0)
- added EX11: GND, Battlebots:Pico_pth_GND, F.Cu at (159.5, 113.7)
- added EX12: GND, Battlebots:Pico_pth_GND, F.Cu at (141.7, 113.7)
- added EX9: GND, Battlebots:Pico_pth_GND, F.Cu at (150.6, 118.6)
- added R6: 10k, Resistor_SMD:R_0603_1608Metric_Pad0.98x0.95mm_HandSolder, B.Cu at (145.8, 79.5)
- added R7: 100, Resistor_SMD:R_0603_1608Metric_Pad0.98x0.95mm_HandSolder, B.Cu at (154.2, 77.5)
- added R8: 10k, Resistor_SMD:R_0603_1608Metric_Pad0.98x0.95mm_HandSolder, B.Cu at (146.2, 103.5)
- added R9: 100, Resistor_SMD:R_0603_1608Metric_Pad0.98x0.95mm_HandSolder, B.Cu at (154.1, 101.6)
- added U3: H3LIS331DLTR, Package_LGA:LGA-16_3x3mm_P0.5mm_LayoutBorder3x5y, B.Cu at (150.6, 81.0)
- D4: renamed from D3; value D_Zener -> Zener Diode; footprint Diode_SMD:D_MicroSMP_KA -> Battlebots:SGP1610N2
- D5: renamed from D4; value D_Zener -> Zener Diode; footprint Diode_SMD:D_MicroSMP_KA -> Battlebots:SGP1610N2
- EX5: renamed from EX3; value GP13 -> GPIO13
- EX7: value GPIO21 -> IO21
- Q1: footprint Package_TO_SOT_SMD:SOT-23_Handsoldering -> Package_TO_SOT_SMD:TSOT-23
- R4: renamed from R7; value 100 -> 6.8k
- R5: renamed from R6; value 300 -> 1K
- moved U4 19.3 mm to (150.8, 102.2)
- moved G*** 13.1 mm to (142.0, 92.2)
- moved G*** 10.7 mm to (140.8, 79.2)
- moved C1 10.2 mm to (148.6, 77.0), turned to 45 degrees
- moved C2 4.22 mm to (149.8, 78.3), turned to 45 degrees
- moved R5 3.78 mm to (141.8, 102.0), turned to 0 degrees
- moved U1 3.70 mm to (150.6, 91.5)
- moved R4 3.51 mm to (141.8, 103.5), turned to 180 degrees
- moved TP3 1.19 mm to (140.8, 98.5)
- moved TP4 0.95 mm to (156.9, 103.2)
- moved D5 0.60 mm to (159.2, 75.2), turned to -90 degrees
- moved Q1 0.40 mm to (161.0, 96.3)
- moved D4 0.17 mm to (141.2, 75.2), turned to 90 degrees
- renumbered D6 to D1, D1 to D2, D2 to D3, EX5 to EX1, EX6 to EX2, TP5 to TP1, TP6 to TP2, TP4 to TP3, TP3 to TP4, TP7 to TP5, TP8 to TP6, U3 to U4
Connections:
- A1 pad 10: Net-(A1-GPIO7) -> /Upper INT1
- A1 pad 14: /BATTV -> /I2C1 SDA
- A1 pad 15: unconnected-(A1-GPIO11-Pad15) -> /I2C1 SCL
- A1 pad 24: Net-(A1-GPIO18) -> /Lower INT1
- A1 pad 25: unconnected-(A1-GPIO19-Pad25) -> /Lower INT2
- A1 pad 26: unconnected-(A1-GPIO20-Pad26) -> /Directional LED
- A1 pad 29: /Directional LED -> unconnected-(A1-GPIO22-Pad29)
- A1 pad 31: unconnected-(A1-GPIO26_ADC0-Pad31) -> /BATTV
- A1 pad 9: Net-(A1-GPIO6) -> /Upper INT2
- R4 pad 2: GND -> +BATT
- R5 pad 1: +BATT -> GND
- U4 pad 11: Net-(U3-INT1) -> /Lower INT1
- U4 pad 4: /I2C0 SCL -> /I2C1 SCL
- U4 pad 6: /I2C0 SDA -> /I2C1 SDA
- U4 pad 9: Net-(U3-INT2) -> /Lower INT2
Routing:
- net +3V3: track 20.6 -> 69.9 mm
- net /Upper INT1: track 0.00 -> 22.9 mm, vias 0 -> 1
- net /BATTV: track 4.30 -> 27.1 mm
- net /Upper INT2: track 0.00 -> 19.5 mm, vias 0 -> 1
- net /Lower INT1: track 0.00 -> 15.5 mm, vias 0 -> 1
- net /Lower INT2: track 0.00 -> 13.3 mm, vias 0 -> 1
- net /I2C1 SDA: track 0.00 -> 9.34 mm, vias 0 -> 1
- net /I2C1 SCL: track 0.00 -> 9.33 mm, vias 0 -> 1
- net GND: track 14.7 -> 21.5 mm, vias 62 -> 51
- net Net-(U3-INT1): track 6.01 -> 0.00 mm
- net /Directional LED: track 23.4 -> 28.8 mm
- net Net-(U3-INT2): track 4.79 -> 0.00 mm
- net Net-(A1-GPIO9): track 14.7 -> 10.9 mm
- net Net-(U3-SDO/SA0): track 0.00 -> 3.36 mm
- net Net-(U4-SDO/SA0): track 3.35 -> 0.00 mm
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Other:
- board text added: "Donut of Doom PCB V2"
- board text added: "ELRS"
- board text added: "RX"
- board text added: "TX"
- board text removed: "Donut of Doom PCB V1"
- board text removed: "ELRS Reciever"
- board text removed: "INT1"
